File: cbuffer/kicad/cbuffer_v2/ki.sch (KiCad schematic (older format))
At the start: 41 parts, among them J1 Header_M1x02, J2 Screw_TermB_01x03, J3 Screw_TermB_01x02, J4 Header_F1x02, J4 Header_M1x02, J5 Header_F1x02, J5 Header_M1x02, J6 Header_F1x02, J6 Header_M1x02, Q1 VN0106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

Commit message: cbuffer:  cbuffer_v2/  v2.0  Revise notes and component values.
This is the initial version being constructed now.
Parts:
- R2: value 10k -> 20k
- R6: value 750 -> 470R 0.5W, 10% Carbon
- Rp3: value 10k -> 10k 1%
- Rs: value 1.0 -> 1.0R 5W, 1%, Wirewound
- U2: value LM358 -> TL052
Other:
- note added: "5 mm, 20 mA"
- note added: "Current Buffer: 1 mA/mV, 1.0 A Full Scale, 1.3 kHz lowpass filter"
- note added: "Future:\n TVS Diode on output\n RC snubber on output\n Offset trim"
- note added: "Iled = (VNN - 1.7 V) / R6"
- note added: "Resistors: 1/4 W, 5% Carbon"
- note removed: "Future:\n TVS Diode on output\n RC snubber on output"
- note removed: "Iled = (VPP - 1.7 V) / R6"
Changed lines of the file:
@@
 EESchema Schematic File Version 4
+LIBS:ki-cache
 EELAYER 26 0
 EELAYER END
@@
 Sheet 1 1
 Title "Current Buffer"
-Date "2022-12-23"
+Date "2023-04-08"
 Rev "v2.0"
 Comp "William A. Hudson"
@@
 P 7400 5250
 F 0 "Rs" H 7332 5204 50  0000 R CNN
-F 1 "1.0" H 7332 5295 50  0000 R CNN
+F 1 "1.0R  5W, 1%, Wirewound" H 7332 5295 50  0000 R CNN
 F 2 "" V 7440 5240 50  0001 C CNN
 F 3 "~" H 7400 5250 50  0001 C CNN
@@
 Current Limit
 Text Notes 5300 6350 0    50   ~ 0
-Future:\n    TVS Diode on output\n    RC snubber on output
+Future:\n    TVS Diode on output\n    RC snubber on output\n    Offset trim
 Connection ~ 7200 3000
 Connection ~ 7400 5000
@@
 P 8600 2250
 F 0 "R6" H 8532 2204 50  0000 R CNN
-F 1 "750" H 8532 2295 50  0000 R CNN
+F 1 "470R 0.5W, 10% Carbon" H 8532 2295 50  0000 R CNN
 F 2 "" V 8640 2240 50  0001 C CNN
 F 3 "~" H 8600 2250 50  0001 C CNN
@@
 	6950 3350 6950 3400
 Wire Wire Line
-	6700 2000 8600 2000
-Wire Wire Line
 	8600 2000 8600 2100
 Wire Wire Line
@@
 Text Notes 9800 5450 0    50   ~ 0
 Output Shunt:
-Text Notes 7700 5350 0    50   ~ 0
+Text Notes 7500 5550 0    50   ~ 0
 Current Sense\nResistor
 Text Notes 8700 2100 0    50   ~ 0
-Iled = (VPP - 1.7 V) / R6
+Iled = (VNN - 1.7 V) / R6
 Text Notes 2600 7100 0    50   ~ 0
 Ilim = 15000 * (4.75 V) / (13750 ohm + Rlim)\n\n
@@
 P 4300 2900
 F 0 "U2" H 4500 3100 50  0000 C CNN
-F 1 "LM358" H 4550 3200 50  0000 C CNN
+F 1 "TL052" H 4550 3200 50  0000 C CNN
 F 2 "" H 4300 2900 50  0001 C CNN
 F 3 "http://www.ti.com/lit/ds/symlink/lm2904-n.pdf" H 4300 2900 50  0001 C CNN
@@
 P 4300 1400
 F 0 "U2" H 4450 1600 50  0000 C CNN
-F 1 "LM358" H 4500 1700 50  0000 C CNN
+F 1 "TL052" H 4500 1700 50  0000 C CNN
 F 2 "" H 4300 1400 50  0001 C CNN
 F 3 "http://www.ti.com/lit/ds/symlink/lm2904-n.pdf" H 4300 1400 50  0001 C CNN
@@
 P 3650 3000
 F 0 "R2" V 3445 3000 50  0000 C CNN
-F 1 "10k" V 3536 3000 50  0000 C CNN
+F 1 "20k" V 3536 3000 50  0000 C CNN
 F 2 "" V 3690 2990 50  0001 C CNN
 F 3 "~" H 3650 3000 50  0001 C CNN
@@
 P 4950 2900
 F 0 "Rp3" V 4745 2900 50  0000 C CNN
-F 1 "10k" V 4836 2900 50  0000 C CNN
+F 1 "10k 1%" V 4836 2900 50  0000 C CNN
 F 2 "" V 4990 2890 50  0001 C CNN
 F 3 "~" H 4950 2900 50  0001 C CNN
@@
 Text Notes 8200 3750 0    50   ~ 0
 no load
+$Comp
+L _Local:GND #PWR?
+U 1 1 63CDC7E0
+P 8300 2000
+F 0 "#PWR?" H 8300 1750 50  0001 C CNN
+F 1 "GND" H 8300 1827 50  0000 C CNN
+F 2 "" H 8200 1650 50  0001 C CNN
+F 3 "" H 8300 1750 50  0001 C CNN
+	1    8300 2000
+	1    0    0    -1
+$EndComp
+Wire Wire Line
+	8600 2000 8300 2000
+Text Notes 9800 2900 0    50   ~ 0
+5 mm, 20 mA
+Text Notes 6300 6700 0    70   ~ 0
+Current Buffer:  1 mA/mV, 1.0 A Full Scale, 1.3 kHz lowpass filter
+Text Notes 2400 7600 0    50   ~ 0
+Resistors:  1/4 W, 5% Carbon
 $EndSCHEMATC

Commit message: cbuffer:  cbuffer_v2/  v2.0.1  Correct NMOS pinout.  Label LED terminals.
Parts:
- Q1: symbol Device:Q_NMOS_GDS -> Device:Q_NMOS_SGD
Other:
- note added: "A"
- note added: "C"
Changed lines of the file:
@@
 Sheet 1 1
 Title "Current Buffer"
-Date "2023-04-08"
-Rev "v2.0"
+Date "2023-04-19"
+Rev "v2.0.1"
 Comp "William A. Hudson"
 Comment1 ""
@@
 Connection ~ 7400 5000
 $Comp
-L Device:Q_NMOS_GDS Q1
+L Device:Q_NMOS_SGD Q1
 U 1 1 639D8B60
 P 8200 2600
@@
 Text Notes 2400 7600 0    50   ~ 0
 Resistors:  1/4 W, 5% Carbon
+Text Notes 8650 2700 0    50   ~ 0
+A
+Text Notes 8650 2800 0    50   ~ 0
+C
 $EndSCHEMATC

Commit message: cbuffer:  kicad/cbuffer_v2  v2.1.0  2023-04-22
    Schematic add Schottky diodes D2, D3 for output back EMF protection.
    BOM minor revisions for as-built.
    Add Schematic Overview to architecture.text.
Parts:
- added D2, D3: SB240, symbol Device:D_Schottky_Small_ALT
- Rs: value 1.0R 5W, 1%, Wirewound -> 1.0R 5W, 5%, Wirewound
Connections:
- net VNN: now also D3.2 (A)
- net VPP: now also D2.1 (K)
- net Vo: now also D2.2 (A), D3.1 (K)
Other:
- note added: "Ho"
- note added: "Lo"
- note added: "Output back EMF\nprotection"
Changed lines of the file:
@@
 Sheet 1 1
 Title "Current Buffer"
-Date "2023-04-19"
-Rev "v2.0.1"
+Date "2023-04-22"
+Rev "v2.1.0"
 Comp "William A. Hudson"
-Comment1 ""
+Comment1 "v2.1  output back EMF protection D2,D3"
 Comment2 ""
 Comment3 ""
@@
 P 7400 5250
 F 0 "Rs" H 7332 5204 50  0000 R CNN
-F 1 "1.0R  5W, 1%, Wirewound" H 7332 5295 50  0000 R CNN
+F 1 "1.0R  5W, 5%, Wirewound" H 7332 5295 50  0000 R CNN
 F 2 "" V 7440 5240 50  0001 C CNN
 F 3 "~" H 7400 5250 50  0001 C CNN
@@
 Connection ~ 6700 2650
 Wire Wire Line
-	7400 3000 7400 4800
+	7400 3000 7400 4500
 $Comp
 L _Local:GND #PWR0104
@@
 	9200 4900 9200 5500
 Wire Wire Line
-	7400 4800 8700 4800
-Wire Wire Line
 	7400 5000 8700 5000
 Wire Wire Line
@@
 Text Notes 9850 4200 0    50   ~ 0
 Rlim    Ilim\n129k    0.5 A\n57.6k   1.0 A\n20.0k   2.1 A\n14.7k   2.5 A
-Text Notes 5300 5800 0    50   ~ 0
+Text Notes 5500 5150 0    50   ~ 0
 Stability Compensation:  Cf4, Rf4, Rf5
 Text Notes 2600 6900 0    50   ~ 0
@@
 Text Notes 8650 2800 0    50   ~ 0
 C
+$Comp
+L Device:D_Schottky_Small_ALT D2
+U 1 1 64440762
+P 7600 4400
+F 0 "D2" V 7554 4468 50  0000 L CNN
+F 1 "SB240" V 7645 4468 50  0000 L CNN
+F 2 "" V 7600 4400 50  0001 C CNN
+F 3 "~" V 7600 4400 50  0001 C CNN
+	1    7600 4400
+	0    1    1    0
+$EndComp
+$Comp
+L Device:D_Schottky_Small_ALT D3
+U 1 1 6444404A
+P 7600 4600
+F 0 "D3" V 7554 4668 50  0000 L CNN
+F 1 "SB240" V 7645 4668 50  0000 L CNN
+F 2 "" V 7600 4600 50  0001 C CNN
+F 3 "~" V 7600 4600 50  0001 C CNN
+	1    7600 4600
+	0    1    1    0
+$EndComp
+Wire Wire Line
+	7600 4500 8200 4500
+Wire Wire Line
+	8200 4500 8200 4800
+Wire Wire Line
+	8200 4800 8700 4800
+Connection ~ 7600 4500
+$Comp
+L _Local:VNN #PWR?
+U 1 1 6445544B
+P 7600 4700
+F 0 "#PWR?" H 7600 4450 50  0001 C CNN
+F 1 "VNN" H 7617 4527 50  0000 C CNN
+F 2 "" H 7600 4700 50  0001 C CNN
+F 3 "" H 7600 4700 50  0001 C CNN
+	1    7600 4700
+	1    0    0    -1
+$EndComp
+$Comp
+L _Local:VPP #PWR?
+U 1 1 644554D4
+P 7600 4300
+F 0 "#PWR?" H 7600 4550 50  0001 C CNN
+F 1 "VPP" H 7617 4473 50  0000 C CNN
+F 2 "" H 7600 4300 50  0001 C CNN
+F 3 "" H 7600 4300 50  0001 C CNN
+	1    7600 4300
+	1    0    0    -1
+$EndComp
+Text Notes 7800 4300 0    50   ~ 0
+Output back EMF\nprotection
+Wire Wire Line
+	7400 4500 7600 4500
+Text Notes 8600 4800 0    50   ~ 0
+Ho
+Text Notes 8600 5000 0    50   ~ 0
+Lo
 $EndSCHEMATC
